Commit message: robot core, gazebo control, joystick

File: description/robot.urdf.xacro (robot description, xacro)
@@ -3,5 +3,5 @@
     <!-- Example link -->
     <xacro:include filename="robot_core.xacro"/>
-        <!-- Example link -->
-    <link name="base_link"></link>
+    <xacro:include filename="properties.xacro"/>
+    <xacro:include filename="gazebo_control.xacro"/>
 </robot>
